File: KiCad/robin.kicad_sch (KiCad schematic)
At the start: 0 parts

Commit message: Added KiCad files
Parts:
- added BT1: Battery_Cell, Battery:BatteryHolder_Keystone_2462_2xAA, symbol Device:Battery_Cell
- added BZ1: Buzzer, Buzzer_Beeper:Buzzer_CUI_CPT-9019S-SMT, symbol Device:Buzzer
- added C1, C2, C3, C4, C5: 100nf, Capacitor_SMD:C_0805_2012Metric_Pad1.18x1.45mm_HandSolder, symbol Device:C
- added C6: 1000uf, Capacitor_THT:CP_Radial_D8.0mm_P5.00mm, symbol Device:C_Polarized
- added D1, D2, D3, D4, D5: SK6812, LED_SMD:LED_SK6812_PLCC4_5.0x5.0mm_P3.2mm, symbol LED:SK6812
- added H1: MountingHole, MountingHole:MountingHole_3mm_Pad_Via, symbol Mechanical:MountingHole
- added J1: Conn_01x06_Male, Connector_PinSocket_2.54mm:PinSocket_2x03_P2.54mm_Vertical, symbol Connector:Conn_01x06_Male
- added R1, R2, R3: 200k, Resistor_SMD:R_0603_1608Metric, symbol Device:R
- added R4, R5: 100k, Resistor_SMD:R_0603_1608Metric, symbol Device:R
- added R6, R7: R, Resistor_SMD:R_0603_1608Metric, symbol Device:R
- added SW4: SW_Push, Button_Switch_SMD:SW_SPST_B3S-1000, symbol Switch:SW_Push
- added U1: ATtiny85-20S, Package_SO:SOIC-8W_5.3x5.3mm_P1.27mm, symbol MCU_Microchip_ATtiny:ATtiny85-20S
- added U2: robin_button, SamacSys_Parts:copp27, symbol xmas:robin_button
Connections:
- new net: D1.2 (DIN), R7.2
- new net: D1.4 (DOUT), D2.2 (DIN)
- new net: D2.4 (DOUT), D3.2 (DIN)
- new net: D3.4 (DOUT), D4.2 (DIN)
- new net: D4.4 (DOUT), D5.2 (DIN)
- new net: BZ1.1 (-), R6.2
- new net GND: BT1.2 (-), BZ1.2 (+), C1.2, C2.2, C3.2, C4.2, C5.2, C6.2, D1.1 (VSS), D2.1 (VSS), D3.1 (VSS), D4.1 (VSS), D5.1 (VSS), J1.6 (Pin_6), SW4.1, U1.4 (GND), U2.1 (gnd)
- new net PB0: J1.4 (Pin_4), R6.1, U1.5 (AREF/PB0)
- new net PB1: J1.3 (Pin_3), R7.1, U1.6 (PB1)
- new net PB2: J1.2 (Pin_2), R1.2, U1.7 (PB2), U2.4 (button3)
- new net PB3: R2.2, U1.2 (XTAL1/PB3), U2.3 (button2)
- new net PB4: R3.2, U1.3 (XTAL2/PB4), U2.2 (button1)
- new net RESET/PB5: J1.5 (Pin_5), R4.2, R5.2, SW4.2, U1.1 (~{RESET}/PB5)
- new net VCC: BT1.1 (+), C1.1, C2.1, C3.1, C4.1, C5.1, C6.1, D1.3 (VDD), D2.3 (VDD), D3.3 (VDD), D4.3 (VDD), D5.3 (VDD), J1.1 (Pin_1), R1.1, R2.1, R3.1, R4.1, R5.1, U1.8 (VCC)
- no-connect marks 0 -> 1
